File: Hardware/Qwiic_USB_Bridge_ATSAMD21G.sch (EAGLE design)
At the start: 24 parts, among them J1 QWIIC_RIGHT_ANGLE, J2 QWIIC_RIGHT_ANGLE, J3 CORTEX_JTAG_DEBUG_MINIMUM_PTH, J6 USB_A_SMT_MALE, U1 3.3V, U2 ATSAMD21G-A, Y1 32.768kHz

Commit message: Updating to build version
Parts:
- removed L1: FB - 30Ohm, SparkFun-Passives:INDUCTOR0603
- added J4: (no value), SparkFun-Connectors:CONN_041X04_NO_SILK
- C10, C11: device samd21-temp:15PF-50V(+-5%)(0402) -> SparkFun-Capacitors:15PF-0603-50V-5%
- C2: device SparkFun-Capacitors:1.0UF-0402-16V-10% -> SparkFun-Capacitors:1.0UF-0603-16V-10%
- C6, C7, C8, C9: device SparkFun-Capacitors:0.1UF-16V(+-10%)(0402) -> SparkFun-Capacitors:0.1UF-0603-25V-(+80/-20%)
- R2: value 10K -> 10k; device SparkFun-Resistors:10KOHM-1/10W-1%(0603)0603 -> SparkFun-Resistors:10KOHM-0603-1/10W-1%
- U2: device samd21-temp:ATSAMD21G-A -> SparkFun-IC-Microcontroller:ATSAMD21G-A
- Y1: device samd21-temp:CRYSTAL3.2X1.5MM -> SparkFun-Clocks:CRYSTAL-32.768KHZSMD-3.2X1.5
Connections:
- removed net VDDANA: C8.1, L1.2, U2.VDDANA
- new net A1: J4.4, U2.A1_PB08(AIN2/SER4:0/TC4:0)
- new net A2: J4.3, U2.A2_PB09(AIN3/SER4:1/TC4:1)
- new net D10: J4.1, U2.PA18(SER1:2+)_D10
- new net D11: J4.2, U2.PA16(I2C/SER1:0+)_D11
- net 3.3V: now also C8.1, U2.VDDANA; no longer L1.1
- net LED_IN: now also U2.PA15(XOUT/SER2:3+)_D5; no longer U2.PA15(XOUT/SER2:3+)
- net SCL: now also U2.PA23(I2C/SER3:0+)_SCL; no longer U2.PA23(I2C/SER3:0+)
- net SDA: now also U2.PA22(I2C/SER3:0+)_SDA; no longer U2.PA22(I2C/SER3:0+)
